Commit message: lab5_3 fixed

File: lab5/ex03/lab5_31/urdf/robot.urdf.xacro (robot description, xacro)
@@ -3,10 +3,10 @@
   <!-- Константы -->
   <xacro:property name="base_length" value="1"/>
-  <xacro:property name="base_width" value="2"/>
+  <xacro:property name="base_width" value="1"/>
   <xacro:property name="base_height" value="0.5"/>
   <xacro:property name="wheel_radius" value="0.3"/>
   <xacro:property name="wheel_length" value="0.2"/>
-  <xacro:property name="wheel_mass" value="2.0"/>
-  <xacro:property name="base_mass" value="10.0"/>
+  <xacro:property name="wheel_mass" value="0.2"/>
+  <xacro:property name="base_mass" value="1.0"/>
   <!-- Базовый корпус робота -->
   <link name="base_link">
@@ -67,5 +67,5 @@
   </link>
     <!-- Левое переднее колесо -->
-  <link name="left_front_wheel">
+  <!--link name="left_front_wheel">
     <visual>
       <geometry>
@@ -84,7 +84,7 @@
       <inertia ixx="0.01" ixy="0.0" ixz="0.0" iyy="0.01" iyz="0.0" izz="0.01"/>
     </inertial>
-  </link>
+  </link-->
   <!-- Правое переднее колесо -->
-  <link name="right_front_wheel">
+  <!--link name="right_front_wheel">
     <visual>
       <geometry>
@@ -103,10 +103,11 @@
       <inertia ixx="0.01" ixy="0.0" ixz="0.0" iyy="0.01" iyz="0.0" izz="0.01"/>
     </inertial>
-  </link>
+  </link-->
   <!-- Соединения для колес -->
   <joint name="left_back_wheel_joint" type="continuous">
     <parent link="base_link"/>
     <child link="left_back_wheel"/>
-    <origin xyz="${base_length/-2 - wheel_length/2} ${base_width/2} 0" rpy="0 ${pi/2*-1} 0"/>
+    <!--origin xyz="${base_length/-2 - wheel_length/2} ${base_width/2} 0" rpy="0 ${pi/2*1} 0"/-->
+    <origin xyz="${base_length/-2 - wheel_length/2} 0 0" rpy="0 ${pi/2*1} 0"/>
     <axis xyz="0 0 1"/>
   </joint>
@@ -114,19 +115,20 @@
     <parent link="base_link"/>
     <child link="right_back_wheel"/>
-    <origin xyz="${base_length/2 + wheel_length/2} ${base_width/2} 0" rpy="0 ${pi/2*1} 0"/>
+    <!--origin xyz="${base_length/2 + wheel_length/2} ${base_width/2} 0" rpy="0 ${pi/2*1} 0"/-->
+    <origin xyz="${base_length/2 + wheel_length/2} 0 0" rpy="0 ${pi/2*1} 0"/>
     <axis xyz="0 0 1"/>
   </joint>
-  <joint name="left_front_wheel_joint" type="continuous">
+  <!--joint name="left_front_wheel_joint" type="continuous">
     <parent link="base_link"/>
     <child link="left_front_wheel"/>
     <origin xyz="${base_length/-2 - wheel_length/2} ${base_width/-2} 0" rpy="0 ${pi/2*-1} 0"/>
     <axis xyz="0 0 1"/>
-  </joint>
-  <joint name="right_front_wheel_joint" type="continuous">
+  </joint-->
+  <!--joint name="right_front_wheel_joint" type="continuous">
     <parent link="base_link"/>
     <child link="right_front_wheel"/>
-    <origin xyz="${base_length/2 + wheel_length/2} ${base_width/-2} 0" rpy="0 ${pi/2*1} 0"/>
+    <origin xyz="${base_length/2 + wheel_length/2} ${base_width/-2} 0" rpy="0 ${pi/2*-1} 0"/>
     <axis xyz="0 0 1"/>
-  </joint>
+  </joint-->
   <!-- Плагин для публикации состояний соединений -->
   <gazebo>
@@ -137,6 +139,6 @@
       <joint_name>left_back_wheel_joint</joint_name>
       <joint_name>right_back_wheel_joint</joint_name>
-      <joint_name>left_front_wheel_joint</joint_name>
-      <joint_name>right_front_wheel_joint</joint_name>
+      <!--joint_name>left_front_wheel_joint</joint_name-->
+      <!--joint_name>right_front_wheel_joint</joint_name-->
     </plugin>
   </gazebo>
@@ -151,5 +153,7 @@
       <left_joint>left_back_wheel_joint</left_joint> <!-- Левое колесо -->
       <right_joint>right_back_wheel_joint</right_joint> <!-- Правое колесо -->
-      <wheel_separation>${base_width}</wheel_separation> <!-- Расстояние между колесами -->
+      <!--left_joint>left_front_wheel_joint</left_joint--> <!-- Левое колесо -->
+      <!--right_joint>right_front_wheel_joint</right_joint--> <!-- Правое колесо -->
+      <wheel_separation>${base_width + wheel_length}</wheel_separation> <!-- Расстояние между колесами -->
       <wheel_diameter>${wheel_radius*2}</wheel_diameter> <!-- Радиус колес -->
       <odometrySource>joint_states</odometrySource> <!-- Источник одометрии -->

Commit message: lab 6 full

File: lab5/ex03/lab5_31/urdf/robot.urdf.xacro (robot description, xacro)
@@ -9,4 +9,10 @@
   <xacro:property name="wheel_mass" value="0.2"/>
   <xacro:property name="base_mass" value="1.0"/>
+  <link name="world"/>
+  <joint name="world_to_base" type="fixed">
+    <parent link="world"/>
+    <child link="base_link"/>
+    <origin xyz="0 0 0" rpy="0 0 0"/>
+  </joint>
   <!-- Базовый корпус робота -->
   <link name="base_link">
@@ -15,5 +21,5 @@
         <box size="${base_length} ${base_width} ${base_height}"/>
       </geometry>
-      <material name="blue"/>
+      <material name="Gazebo/Blue"/>
     </visual>
     <collision>
@@ -34,5 +40,5 @@
         <cylinder length="${wheel_length}" radius="${wheel_radius}"/>
       </geometry>
-      <material name="black"/>
+      <material name="Gazebo/Blue"/>
     </visual>
     <collision>
@@ -53,5 +59,5 @@
         <cylinder length="${wheel_length}" radius="${wheel_radius}"/>
       </geometry>
-      <material name="black"/>
+      <material name="Gazebo/Blue"/>
     </visual>
     <collision>
@@ -66,42 +72,4 @@
     </inertial>
   </link>
-    <!-- Левое переднее колесо -->
-  <!--link name="left_front_wheel">
-    <visual>
-      <geometry>
-        <cylinder length="${wheel_length}" radius="${wheel_radius}"/>
-      </geometry>
-      <material name="black"/>
-    </visual>
-    <collision>
-      <geometry>
-        <cylinder length="${wheel_length}" radius="${wheel_radius}"/>
-      </geometry>
-    </collision>
-    <inertial>
-      <mass value="${wheel_mass}"/>
-      <origin rpy="0 0 0" xyz="0 0 0"/>
-      <inertia ixx="0.01" ixy="0.0" ixz="0.0" iyy="0.01" iyz="0.0" izz="0.01"/>
-    </inertial>
-  </link-->
-  <!-- Правое переднее колесо -->
-  <!--link name="right_front_wheel">
-    <visual>
-      <geometry>
-        <cylinder length="${wheel_length}" radius="${wheel_radius}"/>
-      </geometry>
-      <material name="black"/>
-    </visual>
-    <collision>
-      <geometry>
-        <cylinder length="${wheel_length}" radius="${wheel_radius}"/>
-      </geometry>
-    </collision>
-    <inertial>
-      <mass value="${wheel_mass}"/>
-      <origin rpy="0 0 0" xyz="0 0 0"/>
-      <inertia ixx="0.01" ixy="0.0" ixz="0.0" iyy="0.01" iyz="0.0" izz="0.01"/>
-    </inertial>
-  </link-->
   <!-- Соединения для колес -->
   <joint name="left_back_wheel_joint" type="continuous">
@@ -119,16 +87,4 @@
     <axis xyz="0 0 1"/>
   </joint>
-  <!--joint name="left_front_wheel_joint" type="continuous">
-    <parent link="base_link"/>
-    <child link="left_front_wheel"/>
-    <origin xyz="${base_length/-2 - wheel_length/2} ${base_width/-2} 0" rpy="0 ${pi/2*-1} 0"/>
-    <axis xyz="0 0 1"/>
-  </joint-->
-  <!--joint name="right_front_wheel_joint" type="continuous">
-    <parent link="base_link"/>
-    <child link="right_front_wheel"/>
-    <origin xyz="${base_length/2 + wheel_length/2} ${base_width/-2} 0" rpy="0 ${pi/2*-1} 0"/>
-    <axis xyz="0 0 1"/>
-  </joint-->
   <!-- Плагин для публикации состояний соединений -->
   <gazebo>
@@ -160,3 +116,59 @@
     </plugin>
   </gazebo>
+    <!-- Лидар -->
+  <link name="lidar_link">
+    <visual>
+      <geometry>
+        <cylinder length="0.1" radius="0.05"/>
+      </geometry>
+      <material name="Gazebo/Blue"/>
+    </visual>
+    <collision>
+      <geometry>
+        <cylinder length="0.1" radius="0.05"/>
+      </geometry>
+    </collision>
+    <inertial>
+      <mass value="0.1"/>
+      <origin rpy="0 0 0" xyz="0 0 0"/>
+      <inertia ixx="0.01" ixy="0.0" ixz="0.0" iyy="0.01" iyz="0.0" izz="0.01"/>
+    </inertial  >
+  </link>
+  <joint name="lidar_joint" type="fixed">
+    <parent link="base_link"/>
+    <child link="lidar_link"/>
+    <origin xyz="0 0 0.5" rpy="0 0 0"/>
+  </joint>
+  <gazebo reference="lidar_link">
+    <sensor type="gpu_lidar" name="gpu_lidar">
+      <update_rate>10</update_rate>
+      <ray>
+        <scan>
+          <horizontal>
+            <samples>360</samples>
+            <resolution>1</resolution>
+            <min_angle>-1.57</min_angle>
+            <max_angle>1.57</max_angle>
+          </horizontal>
+        </scan>
+        <range>
+          <min>0.2</min>
+          <max>10.0</max>
+          <resolution>0.01</resolution>
+        </range>
+        <noise>
+          <type>gaussian</type>
+          <mean>0.0</mean>
+          <stddev>0.01</stddev>
+        </noise>
+      </ray>
+      <plugin name="gazebo_ros_laser" filename="libgazebo_ros_gpu_laser.so">
+        <ros>
+          <namespace>/</namespace>
+        </ros>
+        <topicName>/scan</topicName>
+        <frameName>lidar_link</frameName>
+      </plugin>
+    </sensor>
+  </gazebo>
 </robot>
